Commit message: Fix  pioneer 3d

File: sim/rover_description/src/description/pioneer_base.urdf (robot description, URDF)
Before this commit: robot rover, 6 links, 5 joints
Joints:
- joint t_to_b: child base_link -> theta_axis; parent theta_axis -> x_axis
- joint x_to_y: parent x_axis -> theta_axis
- joint y_to_t: child theta_axis -> base_link
