Commit message: fix rotation

File: sim/rover_description/src/description/pioneer_robot1.xacro (robot description, xacro)
@@ -50,5 +50,5 @@
         <child link="theta_axis"/>
         <axis xyz="0 0 1"/>
-        <origin xyz="0.0 0.0 0.0" rpy="${theta} ${theta} ${theta}" />
+        <origin xyz="0.0 0.0 0.0" rpy="0.0 0.0 ${theta}" />
         <limit lower="-3" upper="3" effort="0.5" velocity="0.5"/>
       </joint>

File: sim/rover_description/src/description/pioneer_robot2.xacro (robot description, xacro)
@@ -50,5 +50,5 @@
         <child link="theta_axis"/>
         <axis xyz="0 0 1"/>
-        <origin xyz="0.0 0.0 0.0" rpy="${theta} ${theta} ${theta}" />
+        <origin xyz="0.0 0.0 0.0" rpy="0.0 0.0 ${theta}" />
         <limit lower="-3" upper="3" effort="0.5" velocity="0.5"/>
       </joint>

File: sim/rover_description/src/description/pioneer_robot3.xacro (robot description, xacro)
@@ -50,5 +50,5 @@
         <child link="theta_axis"/>
         <axis xyz="0 0 1"/>
-        <origin xyz="0.0 0.0 0.0" rpy="${theta} ${theta} ${theta}" />
+        <origin xyz="0.0 0.0 0.0" rpy="0.0 0.0 ${theta}" />
         <limit lower="-3" upper="3" effort="0.5" velocity="0.5"/>
       </joint>

File: sim/rover_description/src/description/pioneer_robot4.xacro (robot description, xacro)
@@ -50,5 +50,5 @@
         <child link="theta_axis"/>
         <axis xyz="0 0 1"/>
-        <origin xyz="0.0 0.0 0.0" rpy="${theta} ${theta} ${theta}" />
+        <origin xyz="0.0 0.0 0.0" rpy="0.0 0.0 ${theta}" />
         <limit lower="-3" upper="3" effort="0.5" velocity="0.5"/>
       </joint>

File: sim/rover_description/src/description/pioneer_robot5.xacro (robot description, xacro)
@@ -50,5 +50,5 @@
         <child link="theta_axis"/>
         <axis xyz="0 0 1"/>
-        <origin xyz="0.0 0.0 0.0" rpy="${theta} ${theta} ${theta}" />
+        <origin xyz="0.0 0.0 0.0" rpy="0.0 0.0 ${theta}" />
         <limit lower="-3" upper="3" effort="0.5" velocity="0.5"/>
       </joint>

File: sim/rover_description/src/description/pioneer_robot6.xacro (robot description, xacro)
@@ -50,5 +50,5 @@
         <child link="theta_axis"/>
         <axis xyz="0 0 1"/>
-        <origin xyz="0.0 0.0 0.0" rpy="${theta} ${theta} ${theta}" />
+        <origin xyz="0.0 0.0 0.0" rpy="0.0 0.0 ${theta}" />
         <limit lower="-3" upper="3" effort="0.5" velocity="0.5"/>
       </joint>
