Commit message: Sim

File: install/rover_description/share/rover_description/src/description/pioneer_robot.xacro (robot description, xacro)
@@ -22,7 +22,7 @@
         <visual>
           <xacro:if value="$(arg mesh_enabled)">
-            <origin xyz="-0.1 0.3 -0.5" rpy="0.0 0.0 0.0"/>
+            <origin xyz="0.0 0.0 0.0" rpy="1.57 0.0 1.57"/>
             <geometry>
-              <mesh filename="package://rover_description/meshes/pioneer_3dx.stl"
+              <mesh filename="package://rover_description/meshes/pioneer_cad_v2.stl"
                     scale="0.001 0.001 0.001"/>
             </geometry>
@@ -58,5 +58,5 @@
           <parent link="${robot_id}_base_link"/>
           <child link="${robot_id}_rover_link"/>
-          <origin xyz="0.0 0.0 0.5" rpy="0 0 0" />
+          <origin xyz="0.0 0.0 0.02" rpy="0 0 0" />
           <axis xyz="0 0 0" rpy="0 0 0" />
       </joint>

Commit message: Modify

File: install/rover_description/share/rover_description/src/description/pioneer_robot.xacro (robot description, xacro)
@@ -1,16 +1,15 @@
 <?xml version="1.0"?>
-<robot xmlns:xacro="http://www.ros.org/wiki/xacro" name="multi_rover">
+<robot xmlns:xacro="http://www.ros.org/wiki/xacro" name="pioneer_rover">
   <xacro:arg name="x_pos" default="0.0"/>
   <xacro:arg name="y_pos" default="0.0"/>
   <xacro:arg name="t_pos" default="0.0"/>
-  <xacro:arg name="robot_id" default="p1"/>
   <xacro:arg name="mesh_enabled" default="true"/>
   <link name="world"/>
-  <xacro:macro name="p_instance" params="robot_id x y theta">
-      <link name="${robot_id}_base_link"/>
-      <link name="${robot_id}_x_axis"/>
-      <link name="${robot_id}_y_axis"/>
-      <link name="${robot_id}_theta_axis"/>
-      <link name="${robot_id}_rover_link">
+  <xacro:macro name="p_instance" params="x y theta">
+      <link name="base_link"/>
+      <link name="x_axis"/>
+      <link name="y_axis"/>
+      <link name="theta_axis"/>
+      <link name="rover_link">
         <inertial>
           <origin xyz="0.0 0 0.0" rpy="0 0 0"/>
@@ -30,36 +29,36 @@
         </visual>
       </link>
-      <joint name="${robot_id}_w_to_x" type="prismatic">
+      <joint name="w_to_x" type="prismatic">
         <parent link="world"/>
-        <child link="${robot_id}_x_axis"/>
+        <child link="x_axis"/>
         <axis xyz="1 0 0"/>
         <origin xyz="${x} 0.0 0.0" rpy="0 0 0" />
         <limit lower="-20.0" upper="20.0" effort="0.5" velocity="0.5"/>
       </joint>
-      <joint name="${robot_id}_x_to_y" type="prismatic">
-        <parent link="${robot_id}_theta_axis"/>
-        <child link="${robot_id}_y_axis"/>
+      <joint name="x_to_y" type="prismatic">
+        <parent link="theta_axis"/>
+        <child link="y_axis"/>
         <axis xyz="0 1 0"/>
         <origin xyz="0.0 ${y} 0.0" rpy="0 0 0" />
         <limit lower="-20.0" upper="20.0" effort="0.5" velocity="0.5"/>
       </joint>
-      <joint name="${robot_id}_y_to_t" type="revolute">
-        <parent link="${robot_id}_y_axis"/>
-        <child link="${robot_id}_base_link"/>
+      <joint name="y_to_t" type="revolute">
+        <parent link="y_axis"/>
+        <child link="base_link"/>
         <axis xyz="0 0 1"/>
         <origin xyz="0.0 0.0 0.0" rpy="${theta} ${theta} ${theta}" />
         <limit lower="-3" upper="3" effort="0.5" velocity="0.5"/>
       </joint>
-      <joint name="${robot_id}_t_to_b" type="fixed">
-        <parent link="${robot_id}_x_axis"/>
-        <child link="${robot_id}_theta_axis"/>
+      <joint name="t_to_b" type="fixed">
+        <parent link="x_axis"/>
+        <child link="theta_axis"/>
       </joint>
-      <joint name = "${robot_id}_base_joint"  type = "fixed">
-          <parent link="${robot_id}_base_link"/>
-          <child link="${robot_id}_rover_link"/>
+      <joint name = "base_joint"  type = "fixed">
+          <parent link="base_link"/>
+          <child link="rover_link"/>
           <origin xyz="0.0 0.0 0.02" rpy="0 0 0" />
           <axis xyz="0 0 0" rpy="0 0 0" />
       </joint>
   </xacro:macro>
-  <xacro:p_instance robot_id="$(arg robot_id)" x="$(arg x_pos)" y="$(arg y_pos)" theta="$(arg t_pos)"/>
+  <xacro:p_instance x="$(arg x_pos)" y="$(arg y_pos)" theta="$(arg t_pos)"/>
 </robot>
