Commit message: Fix Bug

File: install/rover_description/share/rover_description/src/description/pioneer_multi_robot.xacro (robot description, xacro)
@@ -39,5 +39,6 @@
         <parent link="p${id}_theta_axis"/>
         <child link="p${id}_y_axis"/>
-        <axis xyz="0 ${y} 0"/>
+        <axis xyz="0 1 0"/>
+        <origin xyz="0.0 ${y} 0.0" rpy="0 0 0" />
         <limit lower="-20.0" upper="20.0" effort="0.5" velocity="0.5"/>
       </joint>

Commit message: Fix Gain

File: install/rover_description/share/rover_description/src/description/pioneer_multi_robot.xacro (robot description, xacro)
@@ -21,5 +21,5 @@
         <visual>
           <xacro:if value="$(arg mesh_enabled)">
-            <origin xyz="0 0 -0.5" rpy="0.0 0.0 0.0"/>
+            <origin xyz="-0.1 0.3 -0.5" rpy="0.0 0.0 0.0"/>
             <geometry>
               <mesh filename="package://rover_description/meshes/pioneer_3dx.stl"

Commit message: update

File: install/rover_description/share/rover_description/src/description/pioneer_multi_robot.xacro (robot description, xacro)
@@ -1,9 +1,7 @@
 <?xml version="1.0"?>
 <robot xmlns:xacro="http://www.ros.org/wiki/xacro" name="multi_rover">
-  <!-- 引数をドキュメント直下で定義 -->
   <xacro:arg name="num_robots" default="3"/>
   <xacro:arg name="mesh_enabled" default="true"/>
   <link name="world"/>
-  <!-- ロボットのインスタンスを定義 -->
   <xacro:macro name="p_instance" params="id x y">
       <link name="p${id}_base_link"/>

File: install/rover_description/share/rover_description/src/description/pioneer_robot.xacro (robot description, xacro)
@@ -13,5 +13,5 @@
       <link name="rover_link">
         <inertial>
-          <origin xyz="0.0 0 0.0" rpy="0 0 0"/>
+          <origin xyz="0.0 0.0 0.0" rpy="0 0 0"/>
           <mass value="3.978"/>
           <inertia ixx="0.021858680" ixy="0.0" ixz="0.010020353"
@@ -37,5 +37,5 @@
       </joint>
       <joint name="x_to_y" type="prismatic">
-        <parent link="theta_axis"/>
+        <parent link="x_axis"/>
         <child link="y_axis"/>
         <axis xyz="0 1 0"/>
@@ -45,5 +45,5 @@
       <joint name="y_to_t" type="revolute">
         <parent link="y_axis"/>
-        <child link="base_link"/>
+        <child link="theta_axis"/>
         <axis xyz="0 0 1"/>
         <origin xyz="0.0 0.0 0.0" rpy="${theta} ${theta} ${theta}" />
@@ -51,6 +51,6 @@
       </joint>
       <joint name="t_to_b" type="fixed">
-        <parent link="x_axis"/>
-        <child link="theta_axis"/>
+        <parent link="theta_axis"/>
+        <child link="base_link"/>
       </joint>
       <joint name = "base_joint"  type = "fixed">
